File: template-pcb/businesscard.kicad_sch (KiCad schematic)
At the start: 39 parts, among them J1 USB_B_Micro, U1 NE555, U2 CD4017

Commit message: layouting and routing of leds
Parts:
- removed C3: 1uf, Capacitor_SMD:C_1206_3216Metric_Pad1.33x1.80mm_HandSolder, symbol Device:CP_Small
- removed J1: USB_B_Micro, Connector_USB:USB_Micro-B_Molex-105017-0001, symbol Connector:USB_B_Micro
- added C2: 1uf, Capacitor_SMD:C_1206_3216Metric_Pad1.33x1.80mm_HandSolder, symbol Device:C
- added J2: USB_C_Receptacle_PowerOnly_4P, usb-c:usb-c-4-pins, symbol Connector:USB_C_Receptacle_PowerOnly_6P
- C1: footprint (none) -> Capacitor_SMD:C_1206_3216Metric_Pad1.33x1.80mm_HandSolder; ALIEXPRESS (none) -> aliexpress.com/item/1005006267002963.html
- D1, D10, D11, D12, D13, D14, D15, D16, D17, D18, D19, D2, D20, D21, D22, D23, D24, D25, D26, D27, D28, D29, D3, D30, D4, D5, D6, D7, D8, D9: ALIEXPRESS (none) -> aliexpress.com/item/1005003327232870.html
- R1, R2, R3: ALIEXPRESS (none) -> aliexpress.com/item/1005007755691325.html
- RV1: ALIEXPRESS (none) -> aliexpress.com/item/1005007368937806.html; MPN (none) -> 3x3 SMD Potentiometer
- U1: ALIEXPRESS (none) -> aliexpress.com/item/1005006748916473.html
- U2: ALIEXPRESS (none) -> aliexpress.com/item/1005009733366256.html
Connections:
- net +5V: now also J2.A9 (VBUS), J2.B9 (VBUS)
- net GND: now also C2.2, J2.A12 (GND), J2.B12 (GND), J2.S1 (SHIELD)
- net Q0: now also U2.3 (Q0)
- net Q1: now also U2.2 (Q1)
- net Q2: now also U2.4 (Q2)
- net Q3: now also U2.7 (Q3)
- net Q4: now also U2.10 (Q4)
- net Q5: now also U2.1 (Q5)
- net Q6: now also U2.5 (Q6)
- net Q7: now also U2.6 (Q7)
- net Q8: now also U2.9 (Q8)
- net Q9: now also U2.11 (Q9)
- net TRIG/TRSH: now also C2.1
- no-connect marks 5 -> 4
